File: 12v1a_psu.kicad_pcb (KiCad board)
At the start: 4 copper layers, 100 x 160 mm, 23 parts, among them J1 AC_IN, J2 P1, J3 P2, J4 Vout, Q1 TIP32AG, U1 L7812

Commit message: Commit to kicad 6, fix libraries
Parts:
- J4: value Vout -> Barrel_Jack
Connections:
- net /S1N renamed Net-(D2-Pad1)
- net /S1P renamed Net-(D1-Pad1)
Routing:
- added copper zone on In1.Cu, net +12V
- added copper zone on In2.Cu, net GND
- removed copper zone on PWR.Cu, net +12V
- removed copper zone on GND.Cu, net GND
Other:
- net class Default removed
